File: pcbs/glove-shield/glove-shield.sch (EAGLE design)
At the start: 19 parts, among them IC1 LM324D, IC2 LM324D, IC3 74LV4053PW

Commit message: Update bom and exported schematics
Parts:
- R27, R28, R4, R5, R6, R7, R8, R9: value (none) -> 15k
Other:
- moved on the sheet: C12

Commit message: Updated glove shield pcb design
Parts:
- removed IC3: 74LV4053PW, toy-mech:74LV4053PW
- added IC4: 4052D, 40xx:4052D
Connections:
- removed net N$29: B1.A2, IC3.3Z
- new net N$1: B1.D13, IC4A.B
- net 5V: now also IC4P.VCC; no longer IC3.VCC
- net ADC1: now also IC4A.Y2; no longer IC3.2Y1
- net ADC2: now also IC4A.X1; no longer IC3.2Y0
- net ADC3: now also IC4A.X0; no longer IC3.3Y1
- net ADC4: now also IC4A.Y1; no longer IC3.3Y0
- net ADC5: now also IC4A.Y0; no longer IC3.1Y1
- net ADC6: now also IC4A.X3; no longer IC3.1Y0
- net ADC7: now also IC4A.Y3; no longer B1.A4
- net ADC8: now also IC4A.X2; no longer B1.A3
- net COM: now also IC4A.INH, IC4P.GND, IC4P.VEE; no longer IC3.!, IC3.GND, IC3.VEE
- net N$26: now also IC4A.Y; no longer IC3.2Z
- net N$31: now also IC4A.A; no longer IC3.S1, IC3.S2, IC3.S3
- net N$9: now also IC4A.X; no longer IC3.1Z
Other:
- moved on the sheet: C2
